Commit message: hokuyo utm30 model

File: urdf/imu.urdf.xacro (robot description, xacro)
@@ -41,5 +41,5 @@
     <origin xyz="0 ${width} ${height1 - axel_offset}" rpy="0 0 0"/>
     <axis xyz="0 1 0"/>
-    <dynamics damping="0.7"/>
+    <dynamics damping="0.001"/>
   </joint>
   <!-- Middle Link -->

File: urdf/kinect.urdf.xacro (robot description, xacro)
@@ -37,5 +37,5 @@
   </link>
   <link name="kinect_optical_link">
-      <visual>
+<!--      <visual>
       <origin xyz="0 0 0" rpy="0 0 0"/>
       <geometry>
@@ -43,10 +43,10 @@
       </geometry>
       <material name="orange"/>
-    </visual>
+    </visual>-->
   </link>
   <joint name="optical_joint" type="fixed">
     <parent link="kinect_link"/>
     <child link="kinect_optical_link"/>
-    <origin xyz="0.01 0 0.15" rpy="1.57 0 0"/>
+    <origin xyz="0.01 0 0.15" rpy="0.0 0 0"/>
   </joint>
   <material name="orange">
@@ -87,5 +87,5 @@
           <frameName>kinect_link</frameName>
           <pointCloudCutoff>0.05</pointCloudCutoff>
-          <rangeMax>4.0</rangeMax>
+          <rangeMax>8.0</rangeMax>
         </plugin>
       </sensor>

Commit message: Updated joints configuration for control

File: urdf/imu.urdf.xacro (robot description, xacro)
@@ -41,5 +41,5 @@
     <origin xyz="0 ${width} ${height1 - axel_offset}" rpy="0 0 0"/>
     <axis xyz="0 1 0"/>
-    <dynamics damping="0.001"/>
+    <dynamics damping="0.001" friction="0.1"/>
   </joint>
   <!-- Middle Link -->
@@ -111,3 +111,15 @@
     </plugin>
   </gazebo>
+  <gazebo>
+</gazebo>
+  <transmission name="tran1">
+    <type>transmission_interface/SimpleTransmission</type>
+    <joint name="joint1">
+      <hardwareInterface>hardware_interface/EffortJointInterface</hardwareInterface>
+    </joint>
+    <actuator name="motor1">
+      <hardwareInterface>hardware_interface/EffortJointInterface</hardwareInterface>
+      <mechanicalReduction>1</mechanicalReduction>
+    </actuator>
+  </transmission>
 </robot>

Commit message: ROS2 update

File: urdf/imu.urdf.xacro (robot description, xacro)
@@ -41,5 +41,5 @@
     <origin xyz="0 ${width} ${height1 - axel_offset}" rpy="0 0 0"/>
     <axis xyz="0 1 0"/>
-    <dynamics damping="0.001" friction="0.1"/>
+    <dynamics damping="0.001"/>
   </joint>
   <!-- Middle Link -->
@@ -102,5 +102,6 @@
   </gazebo>
   <gazebo>
-    <plugin name="imu_plugin" filename="libgazebo_ros_imu.so">
+   <sensor>
+    <plugin name="imu_plugin" filename="libgazebo_ros_imu_sensor.so">
       <alwaysOn>true</alwaysOn>
       <bodyName>sensor</bodyName>
@@ -110,15 +111,5 @@
       <updateRate>20.0</updateRate>
     </plugin>
-  <plugin name="gazebo_ros_control" filename="libgazebo_ros_control.so"/>
+    </sensor>
   </gazebo>
-  <transmission name="tran1">
-    <type>transmission_interface/SimpleTransmission</type>
-    <joint name="joint1">
-      <hardwareInterface>hardware_interface/EffortJointInterface</hardwareInterface>
-    </joint>
-    <actuator name="motor1">
-      <hardwareInterface>hardware_interface/EffortJointInterface</hardwareInterface>
-      <mechanicalReduction>1</mechanicalReduction>
-    </actuator>
-  </transmission>
 </robot>
